Commit message: semi working inverse kinematics

File: models/robot.urdf (robot description, URDF)
Before this commit: robot robot, 9 links, 8 joints
Joints:
- joint base_joint: origin xyz=0 0 0.020303769841725453 rpy=0 0 0 -> xyz=0 0 0.020303769841725453 rpy=0 0 3.141592653589793
- joint hand_to_palm: axis -0.004366731022061443 -0.002831682324096644 -0.9999864565259854 -> 0.02932136493777838 0.013284627894376878 0.9994817538203955; limit lower=-1.57 upper=1.57 effort=1000.0 velocity=0.5 -> lower=-1 upper=1 effort=1000.0 velocity=0.5
- joint palm_to_finger1: axis 0.9999636659509562 0.005282434163997176 0.00669049080617512 -> 0.9999636659509562 0.005282434163996985 0.006690490806174676
- joint palm_to_finger2: axis 0.9999447392592433 0.0053016784442164 0.009078030262021475 -> 0.9999447392592433 0.005301678444212667 0.009078030262015035
- joint shoulder_to_elbow: axis -0.004415797754470727 0.9999791806696806 -0.004705205350021608 -> 0.0018827062370635154 -0.9999871581474631 -0.004705205350021725; limit lower=-1.57 upper=1.57 effort=1000.0 velocity=0.5 -> lower=-1 upper=1 effort=1000.0 velocity=0.5
- joint wrist_to_hand: axis -0.004366731022061433 -0.9999596622889342 0.007848914267704843 -> -0.004366731022061437 -0.9999596622889343 0.007848914267704845
